Commit message: added detachable joint

File: src/simple_scara_arm/urdf/myrobot2.urdf (robot description, URDF)
Before this commit: robot simple_scara, 6 links, 5 joints
Links:
- link link3: geometry collision cylinder length=0.08 radius=0.02; visual cylinder length=0.08 radius=0.02
Joints:
- joint joint3: limit lower=0 upper=0.1 effort=100 velocity=0.2 -> lower=0 upper=0.15 effort=100 velocity=0.2
